File: motherboard/pcb_esp.sch (KiCad schematic (older format))
At the start: 27 parts, among them J1 CONN_01X07, J3 CONN_01X17, J4 CONN_01X13, Q1 S8050, Q2 S8050, U1 LP38691, U2 ESP-12E, U3 USB

Commit message: Version rev2 for double-sided etching.
Parts:
- R1, R10, R11, R12, R13, R14: footprint Resistors_SMD:R_1206_HandSoldering -> Resistors_SMD:R_0805_HandSoldering
Changed lines of the file:
@@
 F 0 "R10" H 1220 6747 50  0000 L CNN
 F 1 "220" H 1220 6654 50  0000 L CNN
-F 2 "Resistors_SMD:R_1206_HandSoldering" V 1080 6700 50  0001 C CNN
+F 2 "Resistors_SMD:R_0805_HandSoldering" V 1080 6700 50  0001 C CNN
 F 3 "" H 1150 6700 50  0001 C CNN
 	1    1150 6700
@@
 F 0 "R11" H 1870 6747 50  0000 L CNN
 F 1 "220" H 1870 6654 50  0000 L CNN
-F 2 "Resistors_SMD:R_1206_HandSoldering" V 1730 6700 50  0001 C CNN
+F 2 "Resistors_SMD:R_0805_HandSoldering" V 1730 6700 50  0001 C CNN
 F 3 "" H 1800 6700 50  0001 C CNN
 	1    1800 6700
@@
 F 0 "R12" H 2570 6747 50  0000 L CNN
 F 1 "220" H 2570 6654 50  0000 L CNN
-F 2 "Resistors_SMD:R_1206_HandSoldering" V 2430 6700 50  0001 C CNN
+F 2 "Resistors_SMD:R_0805_HandSoldering" V 2430 6700 50  0001 C CNN
 F 3 "" H 2500 6700 50  0001 C CNN
 	1    2500 6700
@@
 F 0 "R13" H 3220 6747 50  0000 L CNN
 F 1 "220" H 3220 6654 50  0000 L CNN
-F 2 "Resistors_SMD:R_1206_HandSoldering" V 3080 6700 50  0001 C CNN
+F 2 "Resistors_SMD:R_0805_HandSoldering" V 3080 6700 50  0001 C CNN
 F 3 "" H 3150 6700 50  0001 C CNN
 	1    3150 6700
@@
 F 0 "R14" H 3870 6747 50  0000 L CNN
 F 1 "220" H 3870 6654 50  0000 L CNN
-F 2 "Resistors_SMD:R_1206_HandSoldering" V 3730 6700 50  0001 C CNN
+F 2 "Resistors_SMD:R_0805_HandSoldering" V 3730 6700 50  0001 C CNN
 F 3 "" H 3800 6700 50  0001 C CNN
 	1    3800 6700
@@
 F 0 "R1" V 9900 3600 50  0000 L CNN
 F 1 "0" V 9800 3525 50  0000 L CNN
-F 2 "Resistors_SMD:R_1206_HandSoldering" V 9730 3550 50  0001 C CNN
+F 2 "Resistors_SMD:R_0805_HandSoldering" V 9730 3550 50  0001 C CNN
 F 3 "" H 9800 3550 50  0001 C CNN
 	1    9800 3550
